Commit message: カメラ映像をros2トピックと配信させる

File: src/lab_navigation/urdf/diffbot_sim.urdf.xacro (robot description, xacro)
@@ -1,30 +1,36 @@
-<?xml version="1.0"?>
-<robot name="diffbot" xmlns:xacro="http://www.ros.org/wiki/xacro">
+<?xml version='1.0' encoding='UTF-8'?>
+<robot xmlns:xacro="http://www.ros.org/wiki/xacro" name="diffbot">
   <!-- launch から渡される -->
-  <xacro:arg name="use_mock_hardware" default="false" />
+  <xacro:arg name="use_mock_hardware" default="false"/>
   <!-- Material definitions -->
-  <xacro:include
-    filename="$(find ros2_control_demo_description)/diffbot/urdf/diffbot.materials.xacro" />
+  <xacro:include filename="$(find ros2_control_demo_description)/diffbot/urdf/diffbot.materials.xacro"/>
   <!-- 前後に設置する低摩擦の球形支持 -->
   <xacro:macro name="support_ball" params="prefix name x z radius mass">
     <joint name="${prefix}${name}_joint" type="fixed">
-      <parent link="${prefix}base_link" />
-      <child link="${prefix}${name}" />
-      <origin xyz="${x} 0 ${z}" rpy="0 0 0" />
+      <parent link="${prefix}base_link"/>
+      <child link="${prefix}${name}"/>
+      <origin xyz="${x} 0 ${z}" rpy="0 0 0"/>
     </joint>
     <link name="${prefix}${name}">
       <collision>
-        <geometry><sphere radius="${radius}" /></geometry>
+        <geometry>
+          <sphere radius="${radius}"/>
+        </geometry>
       </collision>
       <visual>
-        <geometry><sphere radius="${radius}" /></geometry>
-        <material name="black" />
-      </visual>
-      <inertial>
-        <mass value="${mass}" />
-        <inertia
-          ixx="${2.0 / 5.0 * mass * radius * radius}" ixy="0" ixz="0"
-          iyy="${2.0 / 5.0 * mass * radius * radius}" iyz="0"
-          izz="${2.0 / 5.0 * mass * radius * radius}" />
+        <geometry>
+          <sphere radius="${radius}"/>
+        </geometry>
+        <material name="black"/>
+      </visual>
+      <inertial>
+        <mass value="${mass}"/>
+        <inertia
+          ixx="${2.0 / 5.0 * mass * radius * radius}"
+          ixy="0"
+          ixz="0"
+          iyy="${2.0 / 5.0 * mass * radius * radius}"
+          iyz="0"
+          izz="${2.0 / 5.0 * mass * radius * radius}"/>
       </inertial>
     </link>
@@ -35,72 +41,68 @@
   </xacro:macro>
   <xacro:macro name="diffbot" params="prefix">
-    <!-- base_link は地面から 0.215 m。車体上端は 0.43 m、
-         車体下端は 0.05 m。前後の補助球は床から 1 mm 浮く。 -->
-    <xacro:property name="PI" value="3.1415926535897931" />
+    <!--
+      base_link は地面から 0.215 m。
+      車体上端は 0.43 m。
+      車体下端は 0.05 m。
+      前後の補助球は床から 1 mm 浮く。
+    -->
+    <xacro:property name="PI" value="3.1415926535897931"/>
     <!-- Robot body -->
-    <xacro:property name="base_bottom_raise" value="0.05" />
-    <xacro:property name="base_box_height" value="${base_height - base_bottom_raise}" />
-    <xacro:property name="base_box_center_z" value="${base_bottom_raise / 2}" />
-    <xacro:property name="base_length" value="0.70" />
-    <xacro:property name="base_width"  value="0.60" />
-    <xacro:property name="base_height" value="0.43" />
+    <xacro:property name="base_bottom_raise" value="0.05"/>
+    <xacro:property name="base_box_height" value="${base_height - base_bottom_raise}"/>
+    <xacro:property name="base_box_center_z" value="${base_bottom_raise / 2}"/>
+    <xacro:property name="base_length" value="0.70"/>
+    <xacro:property name="base_width" value="0.60"/>
+    <xacro:property name="base_height" value="0.43"/>
     <!-- Placeholder body mass -->
-    <xacro:property name="base_mass" value="0.3" />
+    <xacro:property name="base_mass" value="0.3"/>
     <!-- Wheels -->
-    <xacro:property name="wheel_mass" value="0.3" />
-    <xacro:property name="wheel_len" value="0.10" />
-    <xacro:property name="wheel_radius" value="0.135" />
-    <xacro:property name="wheel_separation" value="0.53" />
-    <!-- 駆動輪を主な接地点にし、前後の傾きを補助球で支える。 -->
-    <xacro:property name="support_radius" value="0.03" />
-    <xacro:property name="support_mass" value="0.02" />
-    <xacro:property name="support_x" value="0.25" />
-    <xacro:property name="support_ground_clearance" value="0.001" />
+    <xacro:property name="wheel_mass" value="0.3"/>
+    <xacro:property name="wheel_len" value="0.10"/>
+    <xacro:property name="wheel_radius" value="0.135"/>
+    <xacro:property name="wheel_separation" value="0.53"/>
+    <!-- 駆動輪を主な接地点にし、前後の傾きを補助球で支える -->
+    <xacro:property name="support_radius" value="0.03"/>
+    <xacro:property name="support_mass" value="0.02"/>
+    <xacro:property name="support_x" value="0.25"/>
+    <xacro:property name="support_ground_clearance" value="0.001"/>
     <!-- VLP-16 -->
-    <xacro:property name="vlp_bottom_height_from_ground" value="0.43" />
-    <xacro:property name="vlp_height" value="0.07" />
-    <!--
-      Coordinate assumptions:
-      - base_link remains at its original height of 0.215 m above ground.
-      - The body bottom is 0.05 m above ground; its top stays at 0.43 m.
-      - Wheel center height = wheel radius = 0.135 m above ground.
-      - VLP-16 bottom = 0.43 m above ground.
-      - VLP-16 center = 0.43 + 0.07/2 = 0.465 m above ground.
-    -->
+    <xacro:property name="vlp_bottom_height_from_ground" value="0.43"/>
+    <xacro:property name="vlp_height" value="0.07"/>
     <xacro:property
       name="base_link_height_from_ground"
-      value="${base_height/2}" />
+      value="${base_height/2}"/>
     <xacro:property
       name="wheel_center_z"
-      value="${wheel_radius - base_link_height_from_ground}" />
+      value="${wheel_radius - base_link_height_from_ground}"/>
     <xacro:property
       name="wheel_y"
-      value="${wheel_separation/2}" />
+      value="${wheel_separation/2}"/>
     <xacro:property
       name="support_center_z"
-      value="${support_radius + support_ground_clearance - base_link_height_from_ground}" />
+      value="${support_radius + support_ground_clearance - base_link_height_from_ground}"/>
     <xacro:property
       name="vlp_center_z"
-      value="${vlp_bottom_height_from_ground + vlp_height/2 - base_link_height_from_ground}" />
-    <!-- =========================
+      value="${vlp_bottom_height_from_ground + vlp_height/2 - base_link_height_from_ground}"/>
+    <!-- =========================================================
          Base link
-         ========================= -->
+         ========================================================= -->
     <link name="${prefix}base_link">
       <collision>
-        <origin xyz="0 0 ${base_box_center_z}" rpy="0 0 0" />
-        <geometry>
-          <box size="${base_length} ${base_width} ${base_box_height}" />
+        <origin xyz="0 0 ${base_box_center_z}" rpy="0 0 0"/>
+        <geometry>
+          <box size="${base_length} ${base_width} ${base_box_height}"/>
         </geometry>
       </collision>
       <visual>
-        <origin xyz="0 0 ${base_box_center_z}" rpy="0 0 0" />
-        <geometry>
-          <box size="${base_length} ${base_width} ${base_box_height}" />
-        </geometry>
-        <material name="orange" />
-      </visual>
-      <inertial>
-        <origin xyz="0 0 ${base_box_center_z}" rpy="0 0 0" />
-        <mass value="${base_mass}" />
+        <origin xyz="0 0 ${base_box_center_z}" rpy="0 0 0"/>
+        <geometry>
+          <box size="${base_length} ${base_width} ${base_box_height}"/>
+        </geometry>
+        <material name="orange"/>
+      </visual>
+      <inertial>
+        <origin xyz="0 0 ${base_box_center_z}" rpy="0 0 0"/>
+        <mass value="${base_mass}"/>
         <inertia
           ixx="${base_mass / 12.0 * (base_width*base_width + base_box_height*base_box_height)}"
@@ -109,21 +111,21 @@
           iyy="${base_mass / 12.0 * (base_length*base_length + base_box_height*base_box_height)}"
           iyz="0.0"
-          izz="${base_mass / 12.0 * (base_length*base_length + base_width*base_width)}" />
-      </inertial>
-    </link>
-    <!-- =========================
+          izz="${base_mass / 12.0 * (base_length*base_length + base_width*base_width)}"/>
+      </inertial>
+    </link>
+    <!-- =========================================================
          Left wheel
-         ========================= -->
+         ========================================================= -->
     <joint name="${prefix}left_wheel_joint" type="continuous">
-      <parent link="${prefix}base_link" />
-      <child link="${prefix}left_wheel" />
+      <parent link="${prefix}base_link"/>
+      <child link="${prefix}left_wheel"/>
       <origin
         xyz="0 ${wheel_y} ${wheel_center_z}"
-        rpy="0 0 0" />
-      <axis xyz="0 1 0" />
-      <dynamics damping="0.2" />
+        rpy="0 0 0"/>
+      <axis xyz="0 1 0"/>
+      <dynamics damping="0.2"/>
       <limit
         effort="100"
-        velocity="3.0" />
+        velocity="3.0"/>
     </joint>
     <link name="${prefix}left_wheel">
@@ -131,9 +133,9 @@
         <origin
           xyz="0 0 0"
-          rpy="${PI/2} 0 0" />
+          rpy="${PI/2} 0 0"/>
         <geometry>
           <cylinder
             length="${wheel_len}"
-            radius="${wheel_radius}" />
+            radius="${wheel_radius}"/>
         </geometry>
       </collision>
@@ -141,17 +143,17 @@
         <origin
           xyz="0 0 0"
-          rpy="${PI/2} 0 0" />
+          rpy="${PI/2} 0 0"/>
         <geometry>
           <cylinder
             length="${wheel_len}"
-            radius="${wheel_radius}" />
-        </geometry>
-        <material name="black" />
-      </visual>
-      <inertial>
-        <origin
-          xyz="0 0 0"
-          rpy="${PI/2} 0 0" />
-        <mass value="${wheel_mass}" />
+            radius="${wheel_radius}"/>
+        </geometry>
+        <material name="black"/>
+      </visual>
+      <inertial>
+        <origin
+          xyz="0 0 0"
+          rpy="${PI/2} 0 0"/>
+        <mass value="${wheel_mass}"/>
         <inertia
           ixx="${wheel_mass / 12.0 * (3*wheel_radius*wheel_radius + wheel_len*wheel_len)}"
@@ -160,21 +162,21 @@
           iyy="${wheel_mass / 12.0 * (3*wheel_radius*wheel_radius + wheel_len*wheel_len)}"
           iyz="0.0"
-          izz="${wheel_mass / 2.0 * wheel_radius*wheel_radius}" />
-      </inertial>
-    </link>
-    <!-- =========================
+          izz="${wheel_mass / 2.0 * wheel_radius*wheel_radius}"/>
+      </inertial>
+    </link>
+    <!-- =========================================================
          Right wheel
-         ========================= -->
+         ========================================================= -->
     <joint name="${prefix}right_wheel_joint" type="continuous">
-      <parent link="${prefix}base_link" />
-      <child link="${prefix}right_wheel" />
+      <parent link="${prefix}base_link"/>
+      <child link="${prefix}right_wheel"/>
       <origin
         xyz="0 -${wheel_y} ${wheel_center_z}"
-        rpy="0 0 0" />
-      <axis xyz="0 1 0" />
-      <dynamics damping="0.2" />
+        rpy="0 0 0"/>
+      <axis xyz="0 1 0"/>
+      <dynamics damping="0.2"/>
       <limit
         effort="100"
-        velocity="3.0" />
+        velocity="3.0"/>
     </joint>
     <link name="${prefix}right_wheel">
@@ -182,9 +184,9 @@
         <origin
           xyz="0 0 0"
-          rpy="${PI/2} 0 0" />
+          rpy="${PI/2} 0 0"/>
         <geometry>
           <cylinder
             length="${wheel_len}"
-            radius="${wheel_radius}" />
+            radius="${wheel_radius}"/>
         </geometry>
       </collision>
@@ -192,17 +194,17 @@
         <origin
           xyz="0 0 0"
-          rpy="${PI/2} 0 0" />
+          rpy="${PI/2} 0 0"/>
         <geometry>
           <cylinder
             length="${wheel_len}"
-            radius="${wheel_radius}" />
-        </geometry>
-        <material name="black" />
-      </visual>
-      <inertial>
-        <origin
-          xyz="0 0 0"
-          rpy="${PI/2} 0 0" />
-        <mass value="${wheel_mass}" />
+            radius="${wheel_radius}"/>
+        </geometry>
+        <material name="black"/>
+      </visual>
+      <inertial>
+        <origin
+          xyz="0 0 0"
+          rpy="${PI/2} 0 0"/>
+        <mass value="${wheel_mass}"/>
         <inertia
           ixx="${wheel_mass / 12.0 * (3*wheel_radius*wheel_radius + wheel_len*wheel_len)}"
@@ -211,23 +213,31 @@
           iyy="${wheel_mass / 12.0 * (3*wheel_radius*wheel_radius + wheel_len*wheel_len)}"
           iyz="0.0"
-          izz="${wheel_mass / 2.0 * wheel_radius*wheel_radius}" />
-      </inertial>
-    </link>
-    <!-- 前後の球形補助接地点。旋回中は低摩擦で床を滑る。 -->
-    <xacro:support_ball prefix="${prefix}" name="front_support"
-      x="${support_x}" z="${support_center_z}"
-      radius="${support_radius}" mass="${support_mass}" />
-    <xacro:support_ball prefix="${prefix}" name="rear_support"
-      x="${-support_x}" z="${support_center_z}"
-      radius="${support_radius}" mass="${support_mass}" />
-    <!-- =========================
+          izz="${wheel_mass / 2.0 * wheel_radius*wheel_radius}"/>
+      </inertial>
+    </link>
+    <!-- 前後の球形補助接地点 -->
+    <xacro:support_ball
+      prefix="${prefix}"
+      name="front_support"
+      x="${support_x}"
+      z="${support_center_z}"
+      radius="${support_radius}"
+      mass="${support_mass}"/>
+    <xacro:support_ball
+      prefix="${prefix}"
+      name="rear_support"
+      x="${-support_x}"
+      z="${support_center_z}"
+      radius="${support_radius}"
+      mass="${support_mass}"/>
+    <!-- =========================================================
          Velodyne VLP-16
-         ========================= -->
+         ========================================================= -->
     <joint name="${prefix}scan_joint" type="fixed">
-      <parent link="${prefix}base_link" />
-      <child link="${prefix}velodyne" />
+      <parent link="${prefix}base_link"/>
+      <child link="${prefix}velodyne"/>
       <origin
         xyz="0 0 ${vlp_center_z}"
-        rpy="0 0 0" />
+        rpy="0 0 0"/>
     </joint>
     <link name="${prefix}velodyne">
@@ -236,12 +246,12 @@
         <origin
           xyz="0 0 -0.023"
-          rpy="0 0 0" />
+          rpy="0 0 0"/>
         <geometry>
           <cylinder
             length="0.024"
-            radius="0.052" />
+            radius="0.052"/>
         </geometry>
         <material name="velodyne_black">
-          <color rgba="0.08 0.08 0.08 1.0" />
+          <color rgba="0.08 0.08 0.08 1.0"/>
         </material>
       </visual>
@@ -250,12 +260,12 @@
         <origin
           xyz="0 0 0"
-          rpy="0 0 0" />
+          rpy="0 0 0"/>
         <geometry>
           <cylinder
             length="0.022"
-            radius="0.050" />
+            radius="0.050"/>
         </geometry>
         <material name="velodyne_blue">
-          <color rgba="0.05 0.25 0.55 1.0" />
+          <color rgba="0.05 0.25 0.55 1.0"/>
         </material>
       </visual>
@@ -264,29 +274,27 @@
         <origin
           xyz="0 0 0.023"
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