Commit message: sfm手順のreadmeを追加, urdfの軸方向不整合を解消

File: src/lab_navigation/urdf/diffbot_real.urdf.xacro (robot description, xacro)
@@ -120,5 +120,5 @@
       <parent link="${prefix}base_link" />
       <child link="${prefix}left_wheel" />
-      <origin xyz="0 -${wheel_y} ${wheel_center_z}" rpy="0 0 0" />
+      <origin xyz="0 ${wheel_y} ${wheel_center_z}" rpy="0 0 0" />
       <axis xyz="0 1 0" />
       <dynamics damping="0.2" />
@@ -157,5 +157,5 @@
       <parent link="${prefix}base_link" />
       <child link="${prefix}right_wheel" />
-      <origin xyz="0 ${wheel_y} ${wheel_center_z}" rpy="0 0 0" />
+      <origin xyz="0 -${wheel_y} ${wheel_center_z}" rpy="0 0 0" />
       <axis xyz="0 1 0" />
       <dynamics damping="0.2" />

Commit message: カメラ, imuリンクを追加

File: src/lab_navigation/urdf/diffbot_real.urdf.xacro (robot description, xacro)
@@ -32,6 +32,6 @@
         車輪中心高さ        : 地面から 0.135 m
         base_link 基準の高さ: z = -0.165 m
-        左車輪位置          : y = -0.265 m
-        右車輪位置          : y = +0.265 m
+        左車輪位置          : y = +0.265 m
+        右車輪位置          : y = -0.265 m
       ■ Velodyne VLP-16
         前後位置            : 車体中央（x = 0）
@@ -224,4 +224,25 @@
       </inertial>
     </link>
+    <!-- IMU -->
+    <joint name="${prefix}imu_joint" type="fixed">
+      <parent link="${prefix}base_link"/>
+      <child link="${prefix}imu_link"/>
+      <origin xyz="0.093 0.020 -0.014" rpy="0 0 0"/>
+    </joint>
+    <link name="${prefix}imu_link"/>
+    <!-- Camera physical frame -->
+    <joint name="${prefix}camera_joint" type="fixed">
+      <parent link="${prefix}base_link"/>
+      <child link="${prefix}camera_link"/>
+      <origin xyz="0.290 0.000 0.338" rpy="0 0 0"/>
+    </joint>
+    <link name="${prefix}camera_link"/>
+    <!-- Camera optical frame -->
+    <joint name="${prefix}camera_optical_joint" type="fixed">
+      <parent link="${prefix}camera_link"/>
+      <child link="${prefix}camera_optical_frame"/>
+      <origin xyz="0 0 0" rpy="-${PI/2} 0 -${PI/2}"/>
+    </joint>
+    <link name="${prefix}camera_optical_frame"/>
   </xacro:macro>
   <!-- =========================
